Commit message: updated URDF with joint limits

File: PAROL6_URDF/PAROL6/urdf/PAROL6.urdf (robot description, URDF)
Before this commit: robot PAROL6, 7 links, 6 joints
Links:
- added link world
- link L1: geometry collision mesh filename=package://parol6/meshes/L1.STL; visual mesh filename=package://parol6/meshes/L1.STL
- link L2: geometry collision mesh filename=package://parol6/meshes/L2.STL; visual mesh filename=package://parol6/meshes/L2.STL
- link L3: geometry collision mesh filename=package://parol6/meshes/L3.STL; visual mesh filename=package://parol6/meshes/L3.STL
- link L4: geometry collision mesh filename=package://parol6/meshes/L4.STL; visual mesh filename=package://parol6/meshes/L4.STL
- link L5: geometry collision mesh filename=package://parol6/meshes/L5.STL; visual mesh filename=package://parol6/meshes/L5.STL
- link L6: geometry collision mesh filename=package://parol6/meshes/L6.STL; visual mesh filename=package://parol6/meshes/L6.STL
- link base_link: geometry collision mesh filename=package://parol6/meshes/base_link.STL; visual mesh filename=package://parol6/meshes/base_link.STL
Joints:
- added joint base_joint: type fixed, parent world, child base_link, origin xyz=0.0 0.0 0.00 rpy=0 0 0
- joint L1: limit lower=0 upper=0 effort=0 velocity=0 -> lower=-1.7 upper=1.7 effort=300 velocity=3
- joint L2: limit lower=0 upper=0 effort=0 velocity=0 -> lower=-0.98 upper=1 effort=300 velocity=3
- joint L3: limit lower=0 upper=0 effort=0 velocity=0 -> lower=-2 upper=1.3 effort=300 velocity=3
- joint L4: limit lower=0 upper=0 effort=0 velocity=0 -> lower=-2 upper=2 effort=300 velocity=3
- joint L5: limit lower=0 upper=0 effort=0 velocity=0 -> lower=-2.1 upper=2.1 effort=300 velocity=3
- joint L6: limit lower=0 upper=0 effort=0 velocity=0 -> lower=-3.1 upper=3.1 effort=300 velocity=3
